File: driver_40mm_atmega_v1p9/driver_40mm_atmega.kicad_pcb (KiCad board)
At the start: 6 copper layers, 40.4 x 40.4 mm, 424 parts, among them IC1 ATMEGA328P-M, IC2 ATMEGA328P-M, IC3 ATMEGA328P-M, IC4 ATMEGA328P-M, P1 CONN_2X2, P2 CONN_2X2, P3 CONN_2X2, P4 CONN_2X2, Q1 NMOS, Q10 NMOS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

Commit message: add revision 4
Other:
- board text added: "/G4"
- board text added: "/Modular-LED-Display"
- board text added: "2024-07-29"
- board text added: "BOTTOM"
- board text added: "G4.1 Driver v1.9.4"
- board text added: "LED: XL0402YGC (V : 2…2.1V) R: 240Ω"
- board text added: "f"
- board text added: "https://reiserlab.github.io"
- board text removed: "BOT"
- board text removed: "Panels G4 Driver V1.9R1"
