File: driver_40mm_atmega_v1p9/driver_40mm_atmega.kicad_sch (KiCad schematic)
At the start: 424 parts, among them IC1 ATMEGA328P-M, IC2 ATMEGA328P-M, IC3 ATMEGA328P-M, IC4 ATMEGA328P-M, P1 CONN_2X2, P2 CONN_2X2, P3 CONN_2X2, P4 CONN_2X2, Q1 NMOS, Q10 NMOS, Q11 NMOS, Q12 NMOS, Q13 NMOS, Q14 NMOS, Q15 NMOS, Q16 NMOS, Q2 NMOS, Q3 NMOS, Q4 NMOS, Q5 NMOS, Q6 NMOS, Q7 NMOS, Q8 NMOS, Q9 NMOS, X1 20MHz, X2 20MHz, X3 20MHz, X4 20MHz

Commit message: add revision 4
Parts:
- D1, D10, D100, D101, D102, D103, D104, D105, D106, D107, D108, D109, D11, D110, D111, D112, D113, D114, D115, D116, D117, D118, D119, D12, D120, D121, D122, D123, D124, D125, D126, D127, D128, D129, D13, D130, D131, D132, D133, D134, D135, D136, D137, D138, D139, D14, D140, D141, D142, D143, D144, D145, D146, D147, D148, D149, D15, D150, D151, D152, D153, D154, D155, D156, D157, D158, D159, D16, D160, D161, D162, D163, D164, D165, D166, D167, D168, D169, D17, D170, D171, D172, D173, D174, D175, D176, D177, D178, D179, D18, D180, D181, D182, D183, D184, D185, D186, D187, D188, D189, D19, D190, D191, D192, D193, D194, D195, D196, D197, D198, D199, D2, D20, D200, D201, D202, D203, D204, D205, D206, D207, D208, D209, D21, D210, D211, D212, D213, D214, D215, D216, D217, D218, D219, D22, D220, D221, D222, D223, D224, D225, D226, D227, D228, D229, D23, D230, D231, D232, D233, D234, D235, D236, D237, D238, D239, D24, D240, D241, D242, D243, D244, D245, D246, D247, D248, D249, D25, D250, D251, D252, D253, D254, D255, D256, D26, D27, D28, D29, D3, D30, D31, D32, D33, D34, D35, D36, D37, D38, D39, D4, D40, D41, D42, D43, D44, D45, D46, D47, D48, D49, D5, D50, D51, D52, D53, D54, D55, D56, D57, D58, D59, D6, D60, D61, D62, D63, D64, D65, D66, D67, D68, D69, D7, D70, D71, D72, D73, D74, D75, D76, D77, D78, D79, D8, D80, D81, D82, D83, D84, D85, D86, D87, D88, D89, D9, D90, D91, D92, D93, D94, D95, D96, D97, D98, D99: JLCPCB PN C5160718 -> C9900113976; PN A-SP136G2C-C01-3T -> XL0402YGC
- R10, R11, R12, R13, R14, R15, R16, R17, R18, R19, R20, R21, R22, R23, R24, R25, R26, R27, R28, R29, R30, R31, R32, R33, R34, R35, R36, R5, R6, R7, R8, R9: value 180 -> 240; JLCPCB PN C5141103 -> C166280; PN SC0201F1800G1BNRH -> RTT012430FTH
- R37, R39, R41, R43, R45, R47, R49, R51, R53, R54, R57, R58, R61, R62, R65, R66, R69, R70, R73, R74, R77, R78, R81, R82, R85, R86, R89, R90, R93, R94, R97, R98: JLCPCB PN C2991668 -> C77623; PN RHC-01W1000FT -> RC0201FR-07100RL
Other:
- company: Janelia -> Reiser Lab @ Janelia
- title: G4 Driver 40mm ATMega -> G4.1 Driver 40mm ATMega
